File: pcb/pcb.kicad_pcb (KiCad board)
At the start: 4 copper layers, 185 x 100 mm, 27 parts, among them J1 USB_C_Receptacle, J2 2x20 Header, J3 2x20 Header, SW1 SW_Push, U1 W65C02, U2 28C256, U3 62256, U4 W65C22S, U5 W65C22S, U6 74AC00, U7 74LS04, U8 74LS08, U9 555

Commit message: backup
Parts:
- added C10: 0.1uF, Capacitor_SMD:C_0805_2012Metric, B.Cu at (-78.2, 37.7)
- added C11: 0.1uF, Capacitor_SMD:C_0805_2012Metric, F.Cu at (310.8, -20.1)
- added C12: 0.1uF, Capacitor_SMD:C_0805_2012Metric, F.Cu at (310.8, -17.1)
- added C13: 0.1uF, Capacitor_SMD:C_0805_2012Metric, B.Cu at (-79.0, 48.4)
- added C14: 0.1uF, Capacitor_SMD:C_0805_2012Metric, F.Cu at (315.3, -29.1)
- added C15: 0.1uF, Capacitor_SMD:C_0805_2012Metric, F.Cu at (315.3, -26.1)
- added C16: 0.1uF, Capacitor_SMD:C_0805_2012Metric, F.Cu at (315.3, -20.1)
- added C17: 0.1uF, Capacitor_SMD:C_0805_2012Metric, F.Cu at (354.4, 12.9)
- added C18: 0.1uF, Capacitor_SMD:C_0805_2012Metric, F.Cu at (354.4, 16.0)
- added C19: 0.1uF, Capacitor_SMD:C_0805_2012Metric, F.Cu at (354.4, 19.0)
- added C20: 0.1uF, Capacitor_SMD:C_0805_2012Metric, F.Cu at (354.4, 22.0)
- added C21: 0.1uF, Capacitor_SMD:C_0805_2012Metric, F.Cu at (317.9, 2.34)
- added C22: 0.1uF, Capacitor_SMD:C_0805_2012Metric, F.Cu at (354.4, 28.0)
- added C23: 0.1uF, Capacitor_SMD:C_0805_2012Metric, F.Cu at (354.4, 31.0)
- added C24: 0.1uF, Capacitor_SMD:C_0805_2012Metric, F.Cu at (321.9, 17.5)
- added C25: 0.1uF, Capacitor_SMD:C_0805_2012Metric, F.Cu at (321.9, 20.5)
- added C26: 0.1uF, Capacitor_SMD:C_0805_2012Metric, F.Cu at (277.1, -64.1)
- added C27: 0.1uF, Capacitor_SMD:C_0805_2012Metric, F.Cu at (277.1, -61.1)
- added C28: 0.1uF, Capacitor_SMD:C_0805_2012Metric, F.Cu at (277.1, -58.1)
- added C29: 0.1uF, Capacitor_SMD:C_0805_2012Metric, F.Cu at (277.1, -55.1)
- added C30: 0.1uF, Capacitor_SMD:C_0805_2012Metric, F.Cu at (326.3, 8.44)
- added C31: 0.1uF, Capacitor_SMD:C_0805_2012Metric, F.Cu at (326.3, 11.4)
- added C32: 0.1uF, Capacitor_SMD:C_0805_2012Metric, F.Cu at (341.6, -71.2)
- added C33: 0.1uF, Capacitor_SMD:C_0805_2012Metric, F.Cu at (277.1, -43.0)
- added C34: 0.1uF, Capacitor_SMD:C_0805_2012Metric, F.Cu at (277.1, -40.0)
- added C35: 0.1uF, Capacitor_SMD:C_0805_2012Metric, F.Cu at (281.6, -64.1)
- added C36: 0.1uF, Capacitor_SMD:C_0805_2012Metric, F.Cu at (330.8, -0.59)
- added C37: 0.1uF, Capacitor_SMD:C_0805_2012Metric, F.Cu at (330.8, 2.42)
- added C38: 0.1uF, Capacitor_SMD:C_0805_2012Metric, F.Cu at (358.8, -30.9)
- added C39: 0.1uF, Capacitor_SMD:C_0805_2012Metric, F.Cu at (358.8, -27.9)
- added C40: 0.1uF, Capacitor_SMD:C_0805_2012Metric, F.Cu at (281.6, -49.0)
- added C41: 0.1uF, Capacitor_SMD:C_0805_2012Metric, F.Cu at (281.6, -46.0)
- added C42: 0.1uF, Capacitor_SMD:C_0805_2012Metric, F.Cu at (281.6, -43.0)
- added C43: 0.1uF, Capacitor_SMD:C_0805_2012Metric, F.Cu at (358.8, -15.8)
- added C44: 0.1uF, Capacitor_SMD:C_0805_2012Metric, F.Cu at (363.3, -39.9)
- added C45: 0.1uF, Capacitor_SMD:C_0805_2012Metric, F.Cu at (286.0, -61.1)
- added C46: 0.1uF, Capacitor_SMD:C_0805_2012Metric, F.Cu at (363.3, -33.9)
- added C47: 0.1uF, Capacitor_SMD:C_0805_2012Metric, F.Cu at (363.3, -30.9)
- added C48: 0.1uF, Capacitor_SMD:C_0805_2012Metric, F.Cu at (286.0, -52.0)
- added C49: 0.1uF, Capacitor_SMD:C_0805_2012Metric, F.Cu at (286.0, -49.0)
- added C50: 0.1uF, Capacitor_SMD:C_0805_2012Metric, F.Cu at (315.1, -53.3)
- added C51: 0.1uF, Capacitor_SMD:C_0805_2012Metric, F.Cu at (315.1, -50.3)
- added C52: 0.1uF, Capacitor_SMD:C_0805_2012Metric, F.Cu at (286.0, -40.0)
- added C53: 0.1uF, Capacitor_SMD:C_0805_2012Metric, F.Cu at (290.5, -64.1)
- added C54: 0.1uF, Capacitor_SMD:C_0805_2012Metric, F.Cu at (319.5, -68.3)
- added C55: 0.1uF, Capacitor_SMD:C_0805_2012Metric, F.Cu at (290.5, -58.1)
- added C56: 0.1uF, Capacitor_SMD:C_0805_2012Metric, F.Cu at (290.5, -55.1)
- added C57: 0.1uF, Capacitor_SMD:C_0805_2012Metric, F.Cu at (343.6, -45.0)
- added C58: 0.1uF, Capacitor_SMD:C_0805_2012Metric, F.Cu at (343.6, -42.0)
- added C59: 0.1uF, Capacitor_SMD:C_0805_2012Metric, F.Cu at (343.6, -39.0)
- added C60: 0.1uF, Capacitor_SMD:C_0805_2012Metric, F.Cu at (343.6, -36.0)
- added C8: 0.1uF, Capacitor_SMD:C_0805_2012Metric, F.Cu at (277.5, -83.4)
- added C9: 0.1uF, Capacitor_SMD:C_0805_2012Metric, F.Cu at (310.8, -26.1)
- added H1: MountingHole_Pad, MountingHole:MountingHole_3.2mm_M3_Pad, F.Cu at (25.0, 159.0)
- added H2: MountingHole_Pad, MountingHole:MountingHole_3.2mm_M3_Pad, F.Cu at (215.0, 159.0)
- added H3: MountingHole_Pad, MountingHole:MountingHole_3.2mm_M3_Pad, F.Cu at (25.0, 44.0)
- added H4: MountingHole_Pad, MountingHole:MountingHole_3.2mm_M3_Pad, F.Cu at (215.0, 44.0)
- added J4: 2x03 Header, Connector_IDC:IDC-Header_2x03_P2.54mm_Horizontal, F.Cu at (159.6, 53.2)
- added J5: 2x17 Header, Connector_IDC:IDC-Header_2x20_P2.54mm_Horizontal, F.Cu at (54.1, 53.2)
- added R10: 390, Resistor_SMD:R_0805_2012Metric, F.Cu at (202.4, 62.1)
- added R11: 390, Resistor_SMD:R_0805_2012Metric, F.Cu at (200.3, 58.9)
- added R12: 390, Resistor_SMD:R_0805_2012Metric, F.Cu at (198.1, 61.9)
- added R13: 780, Resistor_SMD:R_0805_2012Metric, F.Cu at (196.3, 58.9)
- added R14: 390, Resistor_SMD:R_0805_2012Metric, F.Cu at (194.6, 61.9)
- added R15: 780, Resistor_SMD:R_0805_2012Metric, F.Cu at (192.3, 58.9)
- added R16: 390, Resistor_SMD:R_0805_2012Metric, F.Cu at (191.0, 61.9)
- added R17: 390, Resistor_SMD:R_0805_2012Metric, F.Cu at (188.6, 58.9)
- added R18: 390, Resistor_SMD:R_0805_2012Metric, F.Cu at (185.8, 62.1)
- added R19: 780, Resistor_SMD:R_0805_2012Metric, F.Cu at (184.6, 58.9)
- added R20: 390, Resistor_SMD:R_0805_2012Metric, F.Cu at (182.3, 62.1)
- added R21: 780, Resistor_SMD:R_0805_2012Metric, F.Cu at (180.7, 58.9)
- added R22: 390, Resistor_SMD:R_0805_2012Metric, F.Cu at (178.7, 62.0)
- added R23: 390, Resistor_SMD:R_0805_2012Metric, F.Cu at (176.9, 58.9)
- added R24: 3K3, Resistor_SMD:R_0805_2012Metric, F.Cu at (-69.6, 43.5)
- added R8: 390, Resistor_SMD:R_0805_2012Metric, F.Cu at (205.8, 62.1)
- added R9: 780, Resistor_SMD:R_0805_2012Metric, F.Cu at (204.5, 58.9)
- added U10: SST39SF010, Package_LCC:PLCC-32_THT-Socket, F.Cu at (76.8, 102.0)
- added U11: W65C51NxP, Package_DIP:DIP-28_W15.24mm_Socket, F.Cu at (171.0, 63.9)
- added U12: 74AC245, Package_SO:TSSOP-20_4.4x6.5mm_P0.65mm, F.Cu at (49.0, 61.5)
- added U13: 74AC245, Package_SO:TSSOP-20_4.4x6.5mm_P0.65mm, F.Cu at (72.3, 61.9)
- added U14: 74AC245, Package_SO:TSSOP-20_4.4x6.5mm_P0.65mm, B.Cu at (49.0, 36.5)
- added U15: 74AC161, Package_SO:SOIC-16_3.9x9.9mm_P1.27mm, F.Cu at (253.2, 125.0)
- added U16: 74AC161, Package_SO:SOIC-16_3.9x9.9mm_P1.27mm, F.Cu at (265.4, 124.9)
- added U17: 74AC04, Package_SO:SOIC-14_3.9x8.7mm_P1.27mm, F.Cu at (-75.0, 131.5)
- added U18: 74AC08, Package_SO:SOIC-14_3.9x8.7mm_P1.27mm, F.Cu at (-66.6, 131.5)
- added U19: 74AC00, Package_SO:SOIC-14_3.9x8.7mm_P1.27mm, F.Cu at (-58.1, 131.5)
- added U20: 74AC161, Package_SO:SOIC-16_3.9x9.9mm_P1.27mm, F.Cu at (253.2, 137.3)
- added U21: 74AC08, Package_SO:SOIC-14_3.9x8.7mm_P1.27mm, F.Cu at (-49.7, 131.5)
- added U22: 74AC161, Package_SO:SOIC-16_3.9x9.9mm_P1.27mm, F.Cu at (265.4, 137.3)
- added U23: 74AC74, Package_SO:SOIC-14_3.9x8.7mm_P1.27mm, F.Cu at (-61.6, 176.8)
- added U24: 74AC74, Package_SO:SOIC-14_3.9x8.7mm_P1.27mm, F.Cu at (-73.1, 176.3)
- added U25: 74AC238, Package_SO:SOIC-16_3.9x9.9mm_P1.27mm, F.Cu at (-84.2, 138.0)
- added U26: 74AC161, Package_SO:SOIC-16_3.9x9.9mm_P1.27mm, F.Cu at (253.2, 149.7)
- added U27: 74AC161, Package_SO:SOIC-16_3.9x9.9mm_P1.27mm, F.Cu at (265.4, 149.7)
- added U28: 74AC245, Package_SO:TSSOP-20_4.4x6.5mm_P0.65mm, F.Cu at (-60.8, 153.7)
- added U29: 74AC08, Package_SO:SOIC-14_3.9x8.7mm_P1.27mm, F.Cu at (214.1, 98.8)
- added U30: 74AC04, Package_SO:SOIC-14_3.9x8.7mm_P1.27mm, F.Cu at (195.4, 98.8)
- added U31: 74AC273, Package_SO:SOIC-20W_7.5x12.8mm_P1.27mm, F.Cu at (-38.4, 174.0)
- added U32: 74AC10, Package_SO:SOIC-14_3.9x8.7mm_P1.27mm, F.Cu at (205.1, 86.1)
- added U33: 74AC20, Package_SO:SOIC-14_3.9x8.7mm_P1.27mm, F.Cu at (204.7, 98.8)
- added U34: 74AC11, Package_SO:SOIC-14_3.9x8.7mm_P1.27mm, F.Cu at (195.4, 111.0)
- added U35: 74AC00, Package_SO:SOIC-14_3.9x8.7mm_P1.27mm, F.Cu at (196.6, 86.1)
- added U36: 74AC08, Package_SO:SOIC-14_3.9x8.7mm_P1.27mm, F.Cu at (-73.2, 153.3)
- added U37: 74AC273, Package_SO:SOIC-20W_7.5x12.8mm_P1.27mm, F.Cu at (-38.3, 136.2)
- added U38: 74AC273, Package_SO:SOIC-20W_7.5x12.8mm_P1.27mm, F.Cu at (-38.3, 154.4)
- added U39: 74AC00, Package_SO:SOIC-14_3.9x8.7mm_P1.27mm, F.Cu at (213.6, 86.1)
- added U40: 74AC574, Package_SO:SOIC-20W_7.5x12.8mm_P1.27mm, F.Cu at (205.4, 72.9)
- added U41: 74AC273, Package_SO:SOIC-20W_7.5x12.8mm_P1.27mm, F.Cu at (-17.5, 136.7)
- added U42: 74AC273, Package_SO:SOIC-20W_7.5x12.8mm_P1.27mm, F.Cu at (-17.5, 154.9)
- added U43: 74AC86, Package_SO:SOIC-14_3.9x8.7mm_P1.27mm, F.Cu at (143.9, 138.7)
- added U44: 74AC283, Package_SO:SOIC-16_3.9x9.9mm_P1.27mm, F.Cu at (118.9, 210.9)
- added U45: 74AC283, Package_SO:SOIC-16_3.9x9.9mm_P1.27mm, F.Cu at (92.0, 210.9)
- added U46: 74AC86, Package_SO:SOIC-14_3.9x8.7mm_P1.27mm, F.Cu at (156.9, 138.7)
- added U47: 74AC283, Package_SO:SOIC-16_3.9x9.9mm_P1.27mm, F.Cu at (109.9, 210.9)
- added U48: 74AC283, Package_SO:SOIC-16_3.9x9.9mm_P1.27mm, F.Cu at (83.0, 210.7)
- added U49: 74AC283, Package_SO:SOIC-16_3.9x9.9mm_P1.27mm, F.Cu at (100.9, 210.9)
- added U50: 74AC283, Package_SO:SOIC-16_3.9x9.9mm_P1.27mm, F.Cu at (74.0, 210.9)
- added U51: 74AC574, Package_SO:SOIC-20W_7.5x12.8mm_P1.27mm, F.Cu at (110.8, 193.4)
- added U52: 74AC574, Package_SO:SOIC-20W_7.5x12.8mm_P1.27mm, F.Cu at (95.5, 193.4)
- added U53: 74AC574, Package_SO:SOIC-20W_7.5x12.8mm_P1.27mm, F.Cu at (150.6, 151.9)
- added U54: 74AC574, Package_SO:SOIC-20W_7.5x12.8mm_P1.27mm, F.Cu at (183.6, 72.9)
- added U55: 74AC157, Package_SO:SOIC-16_3.9x9.9mm_P1.27mm, F.Cu at (143.9, 127.7)
- added U56: 74AC157, Package_SO:SOIC-16_3.9x9.9mm_P1.27mm, F.Cu at (156.9, 127.7)
- added U57: 74AC574, Package_SO:SOIC-20W_7.5x12.8mm_P1.27mm, F.Cu at (150.9, 114.9)
- added U58: 74AC574, Package_SO:SOIC-20W_7.5x12.8mm_P1.27mm, F.Cu at (173.2, 94.8)
- added Y1: 8MHz, Oscillator:Oscillator_SMD_SeikoEpson_SG8002CA-4Pin_7.0x5.0mm, B.Cu at (-54.2, 68.0)
- added Y2: 1.8432MHz, Oscillator:Oscillator_SMD_SeikoEpson_SG8002CA-4Pin_7.0x5.0mm, B.Cu at (-93.4, 41.4)
- added Y3: 25.175MHz, Oscillator:Oscillator_SMD_SeikoEpson_SG8002CA-4Pin_7.0x5.0mm, F.Cu at (-73.1, 89.2)
- C1, C2, C3, C6: value 100nF -> 0.1uF; footprint Capacitor_SMD:C_0805_2012Metric_Pad1.18x1.45mm_HandSolder -> Capacitor_SMD:C_0805_2012Metric; moved to F.Cu
- C4: value 100nF -> 0.1uF; footprint Capacitor_SMD:C_0805_2012Metric_Pad1.18x1.45mm_HandSolder -> Capacitor_SMD:C_0805_2012Metric
- C5: value 100nF -> 10uF; footprint Capacitor_SMD:C_0805_2012Metric_Pad1.18x1.45mm_HandSolder -> Capacitor_THT:C_Radial_D5.0mm_H7.0mm_P2.00mm
- C7: value 100nF -> 0.1uF; footprint Capacitor_SMD:C_0805_2012Metric_Pad1.18x1.45mm_HandSolder -> Capacitor_SMD:C_0805_2012Metric; moved to B.Cu
- J1: value USB_C_Receptacle -> USB_C_Receptacle_USB2.0_16P; footprint Connector_USB:USB_C_Receptacle_Amphenol_12401548E4-2A -> Connector_USB:USB_C_Receptacle_GCT_USB4085
- J2: value 2x20 Header -> VGA Connector; footprint Connector_PinHeader_2.54mm:PinHeader_2x10_P2.54mm_Vertical -> Connector_Dsub:DSUB-15-HD_Socket_Horizontal_P2.29x2.54mm_EdgePinOffset8.35mm_Housed_MountingHolesOffset10.89mm
- J3: value 2x20 Header -> 2x11 Header; footprint Connector_PinHeader_2.54mm:PinHeader_2x10_P2.54mm_Vertical -> Connector_IDC:IDC-Header_2x11_P2.54mm_Horizontal
- R1, R2, R3: footprint Resistor_SMD:R_0805_2012Metric_Pad1.20x1.40mm_HandSolder -> Resistor_SMD:R_0805_2012Metric
- R4: value 3K3 -> 10K; footprint Resistor_SMD:R_0805_2012Metric_Pad1.20x1.40mm_HandSolder -> Resistor_SMD:R_0805_2012Metric; moved to F.Cu
- R5: value 10K -> 3K3; footprint Resistor_SMD:R_0805_2012Metric_Pad1.20x1.40mm_HandSolder -> Resistor_SMD:R_0805_2012Metric
- R6: value 1M -> 3K3; footprint Resistor_SMD:R_0805_2012Metric_Pad1.20x1.40mm_HandSolder -> Resistor_SMD:R_0805_2012Metric
- R7: value 10K -> 3K3; footprint Resistor_SMD:R_0805_2012Metric_Pad1.20x1.40mm_HandSolder -> Resistor_SMD:R_0805_2012Metric; moved to F.Cu
- SW1: footprint Button_Switch_THT:SW_TH_Tactile_Omron_B3F-100x -> Button_Switch_THT:SW_PUSH_6mm
- U1: value W65C02 -> 74AC154; footprint Package_DIP:DIP-40_W15.24mm_Socket -> Package_SO:SOIC-24W_7.5x15.4mm_P1.27mm
- U2: value 28C256 -> 74AC138; footprint Socket:DIP_Socket-28_W11.9mm_W12.7mm_W15.24mm_W17.78mm_W18.5mm_3M_228-1277-00-0602J -> Package_SO:SOIC-16_3.9x9.9mm_P1.27mm
- U3: value 62256 -> 74AC11; footprint Package_DIP:DIP-28_W15.24mm_Socket -> Package_SO:SOIC-14_3.9x8.7mm_P1.27mm
- U4: value W65C22S -> 74AC238; footprint Package_DIP:DIP-40_W15.24mm_Socket -> Package_SO:SOIC-16_3.9x9.9mm_P1.27mm
- U5: value W65C22S -> W65C02
- U6: value 74AC00 -> AS7C256C; footprint Package_DIP:DIP-14_W7.62mm_Socket -> Package_DIP:DIP-28_W7.62mm_Socket
- U7: value 74LS04 -> 7005; footprint Package_DIP:DIP-14_W7.62mm_Socket -> Package_QFP:TQFP-64_14x14mm_P0.8mm
- U8: value 74LS08 -> W65C22S; footprint Package_DIP:DIP-14_W7.62mm_Socket -> Package_DIP:DIP-40_W15.24mm_Socket
- U9: value 555 -> 7005; footprint Package_DIP:DIP-8_W7.62mm -> Package_QFP:TQFP-64_14x14mm_P0.8mm
- moved U7 278.8 mm to (110.2, 174.5)
- moved U8 251.0 mm to (128.8, 63.9), turned to -90 degrees
- moved C1 233.4 mm to (306.4, -32.1), turned to 0 degrees
- moved C4 214.5 mm to (306.4, -23.1), turned to 0 degrees
- moved C3 191.9 mm to (306.4, -26.1)
- moved U6 184.1 mm to (25.0, 109.8), turned to 90 degrees
- moved J2 150.6 mm to (186.7, 52.9), turned to 180 degrees
- moved C2 150.4 mm to (306.4, -29.1)
- moved C5 137.8 mm to (37.3, 50.7)
- moved R7 129.5 mm to (-47.4, 51.8), turned to 180 degrees
- moved U2 120.5 mm to (105.2, 108.4), turned to 0 degrees
- moved C7 116.6 mm to (-47.5, 72.8), turned to 180 degrees
- moved U9 109.3 mm to (151.7, 95.6), turned to -90 degrees
- moved U5 101.0 mm to (24.6, 88.0)
- moved R6 92.7 mm to (-34.7, 46.4), turned to 180 degrees
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Connections:
- C1 pad 1: +5V -> VCC
- C2 pad 1: +5V -> VCC
- C3 pad 1: +5V -> VCC
- C4 pad 1: +5V -> VCC
- C5 pad 1: +5V -> VCC
- C6 pad 1: +5V -> GND
- C6 pad 2: GND -> ~{RES}
- C7 pad 1: Net-(U9-DIS) -> VCC
- J1 pad A4: +5V -> VCC
- J1 pad A9: +5V -> VCC
- J1 pad B4: +5V -> VCC
- J1 pad B9: +5V -> VCC
- J2 pad 1: Net-(U4-PA0) -> /PPU/R
- J2 pad 10: Net-(U4-PB4) -> GND
- J2 pad 11: Net-(U4-PA5) -> unconnected-(J2-Pad11)
- J2 pad 12: Net-(U4-PB5) -> unconnected-(J2-Pad12)
- J2 pad 13: Net-(U4-PA6) -> /PPU/~{HSYNC}
- J2 pad 14: Net-(U4-PB6) -> /PPU/~{VSYNC}
- J2 pad 15: Net-(U4-PA7) -> unconnected-(J2-Pad15)
- J2 pad 2: Net-(U4-PB0) -> /PPU/G
- J2 pad 3: Net-(U4-PA1) -> /PPU/B
- J2 pad 4: Net-(U4-PB1) -> unconnected-(J2-Pad4)
- J2 pad 5: Net-(U4-PA2) -> GND
- J2 pad 6: Net-(U4-PB2) -> GND
- J2 pad 7: Net-(U4-PA3) -> GND
- J2 pad 8: Net-(U4-PB3) -> GND
- J2 pad 9: Net-(U4-PA4) -> unconnected-(J2-Pad9)
- J3 pad 1: Net-(U5-PA0) -> VCC
- J3 pad 10: Net-(U5-PB4) -> Net-(U8-PB6)
- J3 pad 11: Net-(U5-PA5) -> Net-(U8-PA3)
- J3 pad 12: Net-(U5-PB5) -> Net-(U8-PB5)
- J3 pad 13: Net-(U5-PA6) -> Net-(U8-PA2)
- J3 pad 14: Net-(U5-PB6) -> Net-(U8-PB4)
- J3 pad 15: Net-(U5-PA7) -> Net-(U8-PA1)
- J3 pad 16: Net-(U5-PB7) -> Net-(U8-PB3)
- J3 pad 17: Net-(U5-CA1) -> Net-(U8-PA0)
- J3 pad 18: Net-(U5-CB1) -> Net-(U8-PB2)
- J3 pad 19: Net-(U5-CA2) -> Net-(U8-CA2)
- J3 pad 2: Net-(U5-PB0) -> GND
- J3 pad 20: Net-(U5-CB2) -> Net-(U8-PB1)
- J3 pad 3: Net-(U5-PA1) -> Net-(U8-PA7)
- J3 pad 4: Net-(U5-PB1) -> Net-(U8-CB2)
- J3 pad 5: Net-(U5-PA2) -> Net-(U8-PA6)
- J3 pad 6: Net-(U5-PB2) -> Net-(U8-CB1)
- J3 pad 7: Net-(U5-PA3) -> Net-(U8-PA5)
- J3 pad 8: Net-(U5-PB3) -> Net-(U8-PB7)
- J3 pad 9: Net-(U5-PA4) -> Net-(U8-PA4)
- R4 pad 1: Net-(U1-BE) -> VCC
- R4 pad 2: Net-(U1-RDY) -> ~{RES}
- R5 pad 1: +5V -> ~{IRQ}
- R5 pad 2: Net-(U9-TR) -> VCC
- R6 pad 1: +5V -> ~{NMI}
- R6 pad 2: Net-(U9-DIS) -> VCC
- R7 pad 1: +5V -> RDY
- R7 pad 2: ~{NMI} -> VCC
- SW1 pad 2: Net-(U9-TR) -> ~{RES}
- U1 pad 10: /A1 -> unconnected-(U1-S9-Pad10)
- U1 pad 11: /A2 -> unconnected-(U1-S10-Pad11)
- U1 pad 12: /A3 -> GND
- U1 pad 13: /A4 -> unconnected-(U1-S11-Pad13)
- U1 pad 14: /A5 -> unconnected-(U1-S12-Pad14)
- U1 pad 15: /A6 -> unconnected-(U1-S13-Pad15)
- U1 pad 16: /A7 -> unconnected-(U1-S14-Pad16)
- U1 pad 17: /A8 -> unconnected-(U1-S15-Pad17)
- U1 pad 18: /A9 -> GND
- U1 pad 19: /A10 -> GND
- U1 pad 2: Net-(U1-RDY) -> unconnected-(U1-S1-Pad2)
- U1 pad 20: /A11 -> /A15
- U1 pad 21: GND -> /A14
- U1 pad 22: /A12 -> /A13
- U1 pad 23: /A13 -> /A12
- U1 pad 24: /A14 -> VCC
- U1 pad 4: ~{IRQ} -> unconnected-(U1-S3-Pad4)
- U1 pad 6: ~{NMI} -> unconnected-(U1-S5-Pad6)
- U1 pad 7: unconnected-(U1-SYNC-Pad7) -> ~{CS}_{TM}
- U1 pad 8: +5V -> ~{CS}_{IO}
- U1 pad 9: /A0 -> unconnected-(U1-S8-Pad9)
- U2 pad 1: /A14 -> /A13
- U2 pad 10: /A0 -> Net-(U2-O5)
- U2 pad 11: /D0 -> ~{CS}_{EXP}
- U2 pad 12: /D1 -> unconnected-(U2-O3-Pad12)
- U2 pad 13: /D2 -> ~{CS}_{VRAM}
- U2 pad 14: GND -> Net-(U2-O1)
- U2 pad 15: /D3 -> Net-(U2-O0)
- U2 pad 16: /D4 -> VCC
- U2 pad 2: /A12 -> /A14
- U2 pad 3: /A7 -> /A15
- U2 pad 4: /A6 -> GND
- U2 pad 5: /A5 -> GND
- U2 pad 6: /A4 -> VCC
- U2 pad 7: /A3 -> Net-(U2-O7)
- U2 pad 8: /A2 -> GND
- U2 pad 9: /A1 -> Net-(U2-O6)
- U3 pad 1: /A14 -> Net-(U2-O0)
- U3 pad 10: /A0 -> ~{IRQ}_{ACIA}
- U3 pad 11: /D0 -> ~{IRQ}_{VIA}
- U3 pad 12: /D1 -> ~{CS}_{RAM}
- U3 pad 13: /D2 -> VCC
- U3 pad 14: GND -> VCC
- U3 pad 2: /A12 -> Net-(U2-O1)
- U3 pad 3: /A7 -> Net-(U2-O5)
- U3 pad 4: /A6 -> Net-(U2-O6)
- U3 pad 5: /A5 -> Net-(U2-O7)
- U3 pad 6: /A4 -> ~{CS}_{ROM}
- U3 pad 7: /A3 -> GND
- U3 pad 8: /A2 -> Net-(D1-K)
- U3 pad 9: /A1 -> ~{IRQ}_{PPU}
- U4 pad 1: GND -> /A4
- U4 pad 10: Net-(U4-PB0) -> unconnected-(U4-Y5-Pad10)
- U4 pad 11: Net-(U4-PB1) -> unconnected-(U4-Y4-Pad11)
- U4 pad 12: Net-(U4-PB2) -> unconnected-(U4-Y3-Pad12)
- U4 pad 13: Net-(U4-PB3) -> CS_{PPU}
- U4 pad 14: Net-(U4-PB4) -> CS_{ACIA}
- U4 pad 15: Net-(U4-PB5) -> CS_{VIA}
- U4 pad 16: Net-(U4-PB6) -> VCC
- U4 pad 2: Net-(U4-PA0) -> /A5
- U4 pad 3: Net-(U4-PA1) -> /A6
- U4 pad 4: Net-(U4-PA2) -> GND
- U4 pad 5: Net-(U4-PA3) -> GND
- U4 pad 6: Net-(U4-PA4) -> VCC
- U4 pad 7: Net-(U4-PA5) -> unconnected-(U4-Y7-Pad7)
- U4 pad 8: Net-(U4-PA6) -> GND
- U4 pad 9: Net-(U4-PA7) -> unconnected-(U4-Y6-Pad9)
- U5 pad 1: GND -> unconnected-(U5-~{VP}-Pad1)
- U5 pad 10: Net-(U5-PB0) -> /A1
- U5 pad 11: Net-(U5-PB1) -> /A2
- U5 pad 12: Net-(U5-PB2) -> /A3
- U5 pad 13: Net-(U5-PB3) -> /A4
- U5 pad 14: Net-(U5-PB4) -> /A5
- U5 pad 15: Net-(U5-PB5) -> /A6
- U5 pad 16: Net-(U5-PB6) -> /A7
- U5 pad 17: Net-(U5-PB7) -> /A8
- U5 pad 18: Net-(U5-CB1) -> /A9
- U5 pad 19: Net-(U5-CB2) -> /A10
- U5 pad 2: Net-(U5-PA0) -> RDY
- U5 pad 20: +5V -> /A11
- U5 pad 21: ~{IRQ} 1 -> GND
- U5 pad 22: unconnected-(U5-R/~{W}-Pad22) -> /A12
- U5 pad 23: unconnected-(U5-~{CS2}-Pad23) -> /A13
- U5 pad 24: unconnected-(U5-CS1-Pad24) -> /A14
- U5 pad 25: unconnected-(U5-ϕ2-Pad25) -> /A15
- U5 pad 3: Net-(U5-PA1) -> unconnected-(U5-ϕ1-Pad3)
- U5 pad 34: ~{RES} -> R/~{W}
- U5 pad 35: /A3 -> unconnected-(U5-nc-Pad35)
- U5 pad 36: /A2 -> VCC
- U5 pad 37: /A1 -> Net-(U5-ϕ0)
- U5 pad 38: /A0 -> VCC
- U5 pad 39: Net-(U5-CA2) -> CLK
- U5 pad 4: Net-(U5-PA2) -> ~{IRQ}
- U5 pad 40: Net-(U5-CA1) -> ~{RES}
- U5 pad 5: Net-(U5-PA3) -> unconnected-(U5-~{ML}-Pad5)
- U5 pad 6: Net-(U5-PA4) -> ~{NMI}
- U5 pad 7: Net-(U5-PA5) -> SYNC
- U5 pad 8: Net-(U5-PA6) -> VCC
- U5 pad 9: Net-(U5-PA7) -> /A0
- U6 pad 1: unconnected-(U6-Pad1) -> /A14
- U6 pad 10: unconnected-(U6-Pad10) -> /A0
- U6 pad 11: unconnected-(U6-Pad11) -> /D0
- U6 pad 12: unconnected-(U6-Pad12) -> /D1
- U6 pad 13: unconnected-(U6-Pad13) -> /D2
- U6 pad 14: unconnected-(U6E-VCC-Pad14) -> GND
- U6 pad 2: unconnected-(U6-Pad2) -> /A12
- U6 pad 3: unconnected-(U6-Pad3) -> /A7
- U6 pad 4: unconnected-(U6-Pad4) -> /A6
- U6 pad 5: unconnected-(U6-Pad5) -> /A5
- U6 pad 6: unconnected-(U6-Pad6) -> /A4
- U6 pad 7: unconnected-(U6E-GND-Pad7) -> /A3
- U6 pad 8: unconnected-(U6-Pad8) -> /A2
- U6 pad 9: unconnected-(U6-Pad9) -> /A1
- U7 pad 1: unconnected-(U7-Pad1) -> /D2
- U7 pad 10: unconnected-(U7-Pad10) -> /VMD0
- U7 pad 11: unconnected-(U7-Pad11) -> /VMD1
- U7 pad 12: unconnected-(U7-Pad12) -> /VMD2
- U7 pad 13: unconnected-(U7-Pad13) -> VCC
- U7 pad 14: unconnected-(U7G-VCC-Pad14) -> /VMD3
- U7 pad 2: unconnected-(U7-Pad2) -> /D3
- U7 pad 3: unconnected-(U7-Pad3) -> /D4
- U7 pad 4: unconnected-(U7-Pad4) -> /D5
- U7 pad 5: unconnected-(U7-Pad5) -> GND
- U7 pad 6: unconnected-(U7-Pad6) -> /D6
- U7 pad 7: unconnected-(U7G-GND-Pad7) -> /D7
- U7 pad 8: unconnected-(U7-Pad8) -> VCC
- U7 pad 9: unconnected-(U7-Pad9) -> GND
- U8 pad 1: unconnected-(U8-Pad1) -> GND
- U8 pad 10: unconnected-(U8-Pad10) -> Net-(U8-PB0)
- U8 pad 11: unconnected-(U8-Pad11) -> Net-(U8-PB1)
- U8 pad 12: unconnected-(U8-Pad12) -> Net-(U8-PB2)
- U8 pad 13: unconnected-(U8-Pad13) -> Net-(U8-PB3)
- U8 pad 14: unconnected-(U8E-VCC-Pad14) -> Net-(U8-PB4)
- U8 pad 2: unconnected-(U8-Pad2) -> Net-(U8-PA0)
- U8 pad 3: unconnected-(U8-Pad3) -> Net-(U8-PA1)
- U8 pad 4: unconnected-(U8-Pad4) -> Net-(U8-PA2)
- U8 pad 5: unconnected-(U8-Pad5) -> Net-(U8-PA3)
- U8 pad 6: unconnected-(U8-Pad6) -> Net-(U8-PA4)
- U8 pad 7: unconnected-(U8E-GND-Pad7) -> Net-(U8-PA5)
- U8 pad 8: unconnected-(U8-Pad8) -> Net-(U8-PA6)
- U8 pad 9: unconnected-(U8-Pad9) -> Net-(U8-PA7)
- U9 pad 1: GND -> /TMD5
- U9 pad 2: Net-(U9-TR) -> /TMD4
- U9 pad 3: ~{RES} -> /TMD3
- U9 pad 4: unconnected-(U9-R-Pad4) -> /TMD2
- U9 pad 5: unconnected-(U9-CV-Pad5) -> GND
- U9 pad 6: Net-(U9-DIS) -> /TMD1
- U9 pad 7: Net-(U9-DIS) -> /TMD0
- U9 pad 8: +5V -> VCC
Routing:
- net Net-(U29-Pad11): track 0.00 -> 47.3 mm, vias 0 -> 3
- net Net-(U30-Pad6): track 0.00 -> 39.9 mm, vias 0 -> 2
- net Net-(U55-I1b): track 0.00 -> 35.9 mm, vias 0 -> 2
- net Net-(U55-I1a): track 0.00 -> 33.7 mm, vias 0 -> 3
- net /PPU/VC3: track 0.00 -> 33.0 mm, vias 0 -> 2
- net Net-(U55-I0a): track 0.00 -> 32.6 mm, vias 0 -> 2
- net /PPU/~{HSYNC}: track 0.00 -> 31.7 mm
- net Net-(U29-Pad3): track 0.00 -> 31.3 mm, vias 0 -> 4
- net Net-(U30-Pad8): track 0.00 -> 30.8 mm, vias 0 -> 2
- net /PPU/~{VSYNC}: track 0.00 -> 30.5 mm
- net Net-(U55-I0b): track 0.00 -> 28.2 mm, vias 0 -> 3
- net /PPU/VC2: track 0.00 -> 27.6 mm, vias 0 -> 2
- net Net-(U55-I1c): track 0.00 -> 24.2 mm, vias 0 -> 2
- net Net-(U16-~{MR}): track 0.00 -> 22.5 mm, vias 0 -> 2
- net Net-(U33-Pad6): track 0.00 -> 20.8 mm
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- added copper zone on B.Cu, net GND
- added copper zone on F.Cu, net GND
- added copper zone on In2.Cu, net GND
- added copper zone on In3.Cu, net GND
- added copper zone on In4.Cu, net VCC
- removed copper zone on In2.Cu, net +5V
Other:
- board size 185 x 100 mm -> 200 x 125 mm
- copper layers 4 -> 6
