File: pcb/pcb.kicad_sch (KiCad schematic)
At the start: 0 parts

Commit message: added symbols to schematic
Parts:
- added J1: Conn_01x16_Socket, Connector_PinHeader_1.00mm:PinHeader_1x16_P1.00mm_Vertical, symbol Connector:Conn_01x16_Socket
- added U1: W65C02SxP, Package_DIP:DIP-40_W15.24mm_Socket, symbol PCM_65xx-library:W65C02SxP
- added U2: W65C22SxP, Package_DIP:DIP-40_W15.24mm_Socket, symbol PCM_65xx-library:W65C22SxP
- added U3: 28C256, Package_DIP:DIP-28_W15.24mm_Socket, symbol Memory_EEPROM:28C256
- added U4: HM62256BLP, Package_DIP:DIP-28_W15.24mm_Socket, symbol Memory_RAM:HM62256BLP

Commit message: update
Parts:
- added J2: USB_C_Receptacle, Connector_USB:USB_C_Receptacle_Amphenol_12401548E4-2A, symbol Connector:USB_C_Receptacle
- added R1, R2: 5.11K, symbol Device:R
- added R3: 1M, symbol Device:R
- added U4: 27C512, Package_DIP:DIP-28_W15.24mm_Socket, symbol Memory_EPROM:27C512
- renumbered U4 to U5
Connections:
- net A1: now reaches U1.10 (A1)
- net A1: now also U3.9 (A1), U5.9 (A1)
- net A2: now reaches U1.11 (A2)
- net A2: now also U3.8 (A2), U5.8 (A2)
- net A3: now reaches U1.12 (A3)
- net A3: now also U3.7 (A3), U5.7 (A3)
- net A4: now reaches U1.13 (A4)
- net A4: now also U3.6 (A4), U5.6 (A4)
- net A5: now reaches U1.14 (A5)
- net A5: now also U3.5 (A5), U5.5 (A5)
- net A6: now reaches U1.15 (A6)
- net A6: now also U3.4 (A6), U5.4 (A6)
- net A7: now reaches U1.16 (A7)
- net A7: now also U3.3 (A7), U5.3 (A7)
- net A8: now reaches U1.17 (A8)
- net A8: now also U3.25 (A8), U5.25 (A8)
- net A9: now reaches U1.18 (A9)
- net A9: now also U3.24 (A9), U5.24 (A9)
- net A10: now reaches U1.19 (A10)
- net A10: now also U3.21 (A10), U5.21 (A10)
- net A11: now reaches U1.20 (A11)
- net A11: now also U3.23 (A11), U5.23 (A11)
- net A12: now reaches U1.22 (A12)
- net A12: now also U3.2 (A12), U5.2 (A12)
- net A13: now reaches U1.23 (A13)
- net A13: now also U3.26 (A13), U5.26 (A13)
- net A14: now reaches U1.24 (A14)
- net A14: now also U3.1 (A14), U5.1 (A14)
- net A15: now reaches U1.25 (A15)
- net D7: now reaches U1.26 (D7)
- net D7: now also U2.26 (D7), U3.19 (D7), U5.19 (Q7)
- net D6: now reaches U1.27 (D6)
- net D6: now also U2.27 (D6), U3.18 (D6), U5.18 (Q6)
- net D5: now reaches U1.28 (D5)
- net D5: now also U2.28 (D5), U3.17 (D5), U5.17 (Q5)
- net D4: now reaches U1.29 (D4)
- net D4: now also U2.29 (D4), U3.16 (D4), U5.16 (Q4)
- net D3: now reaches U1.30 (D3)
- net D3: now also U2.30 (D3), U3.15 (D3), U5.15 (Q3)
- net D2: now reaches U1.31 (D2)
- net D2: now also U2.31 (D2), U3.13 (D2), U5.13 (Q2)
- net D1: now reaches U1.32 (D1)
- net D1: now also U2.32 (D1), U3.12 (D1), U5.12 (Q1)
- net D0: now reaches U1.33 (D0)
- net D0: now also U2.33 (D0), U3.11 (D0), U5.11 (Q0)
- net A0: now reaches U1.9 (A0)
- net A0: now also U3.10 (A0), U5.10 (A0)
- new net: J2.A1 (GND), J2.A12 (GND), J2.B1 (GND), J2.B12 (GND)
- new net: J2.A4 (VBUS), J2.A9 (VBUS), J2.B4 (VBUS), J2.B9 (VBUS)
- new net: J2.A5 (CC1), R2.1
- new net: J2.B5 (CC2), R1.1
- new net: J2.S1 (SHIELD), R3.1
- new net GND: R1.2, R2.2, R3.2
- no-connect marks 0 -> 14
Other:
- moved on the sheet: J1, U2, U3

Commit message: lots of updates
Parts:
- removed J1: Conn_01x16_Socket, Connector_PinHeader_1.00mm:PinHeader_1x16_P1.00mm_Vertical, symbol Connector:Conn_01x16_Socket
- removed J2: USB_C_Receptacle, Connector_USB:USB_C_Receptacle_Amphenol_12401548E4-2A, symbol Connector:USB_C_Receptacle
- removed U4: 27C512, Package_DIP:DIP-28_W15.24mm_Socket, symbol Memory_EPROM:27C512
- added J1: USB_C_Receptacle, Connector_USB:USB_C_Receptacle_Amphenol_12401548E4-2A, symbol Connector:USB_C_Receptacle
- added J2, J3, J4, J5: Conn_01x10_Pin, Connector_PinHeader_2.00mm:PinHeader_1x10_P2.00mm_Vertical, symbol Connector:Conn_01x10_Pin
- added J6: Conn_01x02_Pin, Connector_PinHeader_2.00mm:PinHeader_1x02_P2.00mm_Vertical, symbol Connector:Conn_01x02_Pin
- added R4: 1M, Resistor_THT:R_Axial_DIN0207_L6.3mm_D2.5mm_P7.62mm_Horizontal, symbol Device:R
- added SW1: SW_Push, Button_Switch_THT:SW_PUSH-12mm, symbol Switch:SW_Push
- added U10: 74HC04, Package_DIP:DIP-14_W7.62mm_Socket, symbol 74xx:74LS04
- added U3: W65C22SxP, Package_DIP:DIP-40_W15.24mm_Socket, symbol PCM_65xx-library:W65C22SxP
- added U6: 74HC684, Package_DIP:DIP-20_W7.62mm_Socket, symbol Other:74HC684
- added U7, U8: 74HC680, Package_DIP:DIP-20_W7.62mm_Socket, symbol Other:74HC680
- added U9: 74HC00, Package_DIP:DIP-14_W7.62mm_Socket, symbol 74xx:74LS00
- added Y1: MCO-1510A, Oscillator:Oscillator_DIP-14, symbol Other:MCO-1510A
- R1: value 5.11K -> 220; footprint (none) -> Resistor_THT:R_Axial_DIN0207_L6.3mm_D2.5mm_P7.62mm_Horizontal
- R2: footprint (none) -> Resistor_THT:R_Axial_DIN0207_L6.3mm_D2.5mm_P7.62mm_Horizontal
- R3: value 1M -> 5.11K; footprint (none) -> Resistor_THT:R_Axial_DIN0207_L6.3mm_D2.5mm_P7.62mm_Horizontal
- renumbered U3 to U4
Connections:
- net A0: now also U2.38 (RS0), U3.38 (RS0)
- net A1: now also U2.37 (RS1), U3.37 (RS1)
- net A10: now also U6.6 (P2), U7.3 (A2), U8.4 (A3)
- net A11: now also U6.8 (P3), U7.4 (A3), U8.5 (A4)
- net A12: now also U6.11 (P4), U7.5 (A4), U8.6 (A5)
- net A13: now also U6.13 (P5), U7.6 (A5), U8.7 (A6)
- net A14: now also U6.15 (P6), U7.7 (A6), U8.8 (A7)
- net A15: now also U10.1, U6.17 (P7), U7.13 (A11), U8.13 (A11)
- net A2: now also U2.36 (RS2), U3.36 (RS2)
- net A3: now also U2.35 (RS3), U3.35 (RS3)
- net A4: now also U7.8 (A7), U8.1 (A0)
- net A5: now also U7.9 (A8), U8.9 (A8)
- net A6: now also U7.11 (A9), U8.11 (A9)
- net A7: now also U7.12 (A10), U8.12 (A10)
- net A8: now also U6.2 (P0), U7.1 (A0), U8.2 (A1)
- net A9: now also U6.4 (P1), U7.2 (A1), U8.3 (A2)
- net D0: now also U3.33 (D0)
- net D1: now also U3.32 (D1)
- net D2: now also U3.31 (D2)
- net D3: now also U3.30 (D3)
- net D4: now also U3.29 (D4)
- net D5: now also U3.28 (D5)
- net D6: now also U3.27 (D6)
- net D7: now also U3.26 (D7)
- net GND: now also U1.21 (VSS), U2.1 (VSS), U4.14 (GND), U4.22 (~{OE}), U5.14 (GND), U5.22 (~{OE}), J1.A1 (GND), J1.A12 (GND), J1.B1 (GND), J1.B12 (GND), J6.2 (Pin_2), R4.2, SW1.1, U10.7 (GND), U3.1 (VSS), U6.10 (GND), U6.18 (Q7), U7.10 (VSS), U7.17 (P3), U7.19 (C), U8.10 (VSS), U8.14 (P0), U8.15 (P1), U8.16 (P2), U8.19 (C), U9.7 (GND), Y1.7 (GND); no longer R1.2
- net at R2.1: now also J1.B5 (CC2)
- net +5V: now reaches R1.1
- net +5V: now also U1.2 (RDY), U1.36 (BE), U1.38 (~{SO}), U1.6 (~{NMI}), U1.8 (VDD), U2.20 (VCC), U4.27 (~{WE}), U4.28 (VCC), U5.28 (VCC), J1.A4 (VBUS), J1.A9 (VBUS), J1.B4 (VBUS), J1.B9 (VBUS), J6.1 (Pin_1), U10.14 (VCC), U3.20 (VCC), U6.12 (Q4), U6.14 (Q5), U6.16 (Q6), U6.20 (VCC), U6.3 (Q0), U6.5 (Q1), U6.7 (Q2), U6.9 (Q3), U7.14 (P0), U7.15 (P1), U7.16 (P2), U7.20 (VCC), U8.17 (P3), U8.20 (VCC), U9.14 (VCC), Y1.14 (Vcc)
- net at R3.1: now also J1.A5 (CC1)
- net R/~{W}: now reaches U1.34 (R/~{W})
- net R/~{W}: now also U2.22 (R/~{W}), U5.27 (~{WE}), U3.22 (R/~{W})
- net CLK: now reaches U1.37 (ϕ0)
- net CLK: now also U2.25 (ϕ2), U3.25 (ϕ2), U9.2, Y1.8 (OUT)
- net at U1.4 (~{IRQ}): now also U9.8
- net ~{RES}: now reaches U1.40 (~{RES})
- net ~{RES}: now also R1.2, U2.34 (~{RES}), SW1.2, U3.34 (~{RES})
- net at U4.20 (~{CS}): now also U10.2
- net at U5.20 (~{CS}): now also U9.3
- net at U2.10 (PB0): now also J3.1 (Pin_1)
- net at U2.11 (PB1): now also J3.2 (Pin_2)
- net at U2.12 (PB2): now also J3.3 (Pin_3)
- net at U2.13 (PB3): now also J3.4 (Pin_4)
- net at U2.14 (PB4): now also J3.5 (Pin_5)
- net at U2.15 (PB5): now also J3.6 (Pin_6)
- net at U2.16 (PB6): now also J3.7 (Pin_7)
- net at U2.17 (PB7): now also J3.8 (Pin_8)
- net at U2.18 (CB1): now also J3.9 (Pin_9)
- net at U2.19 (CB2): now also J3.10 (Pin_10)
- net at U2.2 (PA0): now also J2.1 (Pin_1)
- net ~{IRQ} 1: now reaches U2.21 (~{IRQ})
- net ~{IRQ} 1: now also U9.4
- net at U2.23 (~{CS2}): now also U10.5, U7.18 (Y)
- net at U2.24 (CS1): now also U10.6
- net at U2.3 (PA1): now also J2.2 (Pin_2)
- net at U2.39 (CA2): now also J2.10 (Pin_10)
- net at U2.4 (PA2): now also J2.3 (Pin_3)
- net at U2.40 (CA1): now also J2.9 (Pin_9)
- net at U2.5 (PA3): now also J2.4 (Pin_4)
- net at U2.6 (PA4): now also J2.5 (Pin_5)
- net at U2.7 (PA5): now also J2.6 (Pin_6)
- net at U2.8 (PA6): now also J2.7 (Pin_7)
- net at U2.9 (PA7): now also J2.8 (Pin_8)
- new net: J5.1 (Pin_1), U3.10 (PB0)
- new net: J5.2 (Pin_2), U3.11 (PB1)
- new net: J5.3 (Pin_3), U3.12 (PB2)
- new net: J5.4 (Pin_4), U3.13 (PB3)
- new net: J5.5 (Pin_5), U3.14 (PB4)
- new net: J5.6 (Pin_6), U3.15 (PB5)
- new net: J5.7 (Pin_7), U3.16 (PB6)
- new net: J5.8 (Pin_8), U3.17 (PB7)
- new net: J5.9 (Pin_9), U3.18 (CB1)
- new net: J5.10 (Pin_10), U3.19 (CB2)
- new net: J4.1 (Pin_1), U3.2 (PA0)
- new net: U10.9, U3.23 (~{CS2}), U8.18 (Y)
- new net: U10.8, U3.24 (CS1)
- new net: J4.2 (Pin_2), U3.3 (PA1)
- new net: J4.10 (Pin_10), U3.39 (CA2)
- new net: J4.3 (Pin_3), U3.4 (PA2)
- new net: J4.9 (Pin_9), U3.40 (CA1)
- new net: J4.4 (Pin_4), U3.5 (PA3)
- new net: J4.5 (Pin_5), U3.6 (PA4)
- new net: J4.6 (Pin_6), U3.7 (PA5)
- new net: J4.7 (Pin_7), U3.8 (PA6)
- new net: J4.8 (Pin_8), U3.9 (PA7)
- new net: J1.S1 (SHIELD), R4.1
- new net: U10.3, U6.1 (~{P>Q})
- new net: U10.4, U9.1
- new net: U9.10, U9.6, U9.9
- new net ~{IRQ} 2: U3.21 (~{IRQ}), U9.5
- no-connect marks 14 -> 20
Other:
- moved on the sheet: U2, U4

Commit message: Finished vesrsion 1 of the project
Parts:
- removed U10: 74HC04, Package_DIP:DIP-14_W7.62mm_Socket, symbol 74xx:74LS04
- removed U6: 74HC684, Package_DIP:DIP-20_W7.62mm_Socket, symbol Other:74HC684
- removed U7, U8: 74HC680, Package_DIP:DIP-20_W7.62mm_Socket, symbol Other:74HC680
- removed unit 1 of U9
- removed unit 2 of U9
- removed unit 3 of U9
- removed Y1: MCO-1510A, Oscillator:Oscillator_DIP-14, symbol Other:MCO-1510A
- added J7: DE15_Socket_HighDensity_MountingHoles, Connector_Dsub:DSUB-15-HD_Socket_Horizontal_P2.29x2.54mm_EdgePinOffset8.35mm_Housed_MountingHolesOffset10.89mm, symbol Connector:DE15_Socket_HighDensity_MountingHoles
- added R10, R6, R8: 680, Resistor_THT:R_Axial_DIN0207_L6.3mm_D2.5mm_P7.62mm_Horizontal, symbol Device:R
- added R11: 3.3K, Resistor_THT:R_Axial_DIN0207_L6.3mm_D2.5mm_P7.62mm_Horizontal, symbol Device:R
- added R5, R7, R9: 1.5K, Resistor_THT:R_Axial_DIN0207_L6.3mm_D2.5mm_P7.62mm_Horizontal, symbol Device:R
- added U10, U11, U12, U13, U8, U9: 74HC161, Package_DIP:DIP-16_W7.62mm_Socket, symbol 74xx:74LS161
- added U14, U21: 74LS08, Package_DIP:DIP-14_W7.62mm_Socket, symbol 74xx:74LS08
- added U15, U20: 74LS10, Package_DIP:DIP-14_W7.62mm_Socket, symbol 74xx:74LS10
- added U16: 74LS04, Package_DIP:DIP-14_W7.62mm_Socket, symbol 74xx:74LS04
- added U17, U19: 74LS00, Package_DIP:DIP-14_W7.62mm_Socket, symbol 74xx:74LS00
- added U18: 74LS20, Package_DIP:DIP-14_W7.62mm_Socket, symbol 74xx:74LS20
- added U22, U23, U24: 74LS245, Package_DIP:DIP-20_W7.62mm_Socket, symbol 74xx:74LS245
- added U25: 74LS32, Package_DIP:DIP-14_W7.62mm_Socket, symbol 74xx:74LS32
- added U7: 74HC04, Package_DIP:DIP-14_W7.62mm_Socket, symbol 74xx:74LS04
- added Y1: 25.175 Mhz, Oscillator:Oscillator_DIP-14, symbol Other:Clock
- renumbered U9 to U6
Connections:
- net A4 is gone; now on net ~{CS}_{VIA A}: U1.13 (A4), U4.6 (A4), U5.6 (A4)
- net +5V: now also U10.16 (VCC), U10.7 (CEP), U10.9 (~{PE}), U11.10 (CET), U11.16 (VCC), U11.7 (CEP), U11.9 (~{PE}), U12.16 (VCC), U12.7 (CEP), U12.9 (~{PE}), U13.16 (VCC), U13.7 (CEP), U13.9 (~{PE}), U14.14 (VCC), U15.14 (VCC), U16.14 (VCC), U17.14 (VCC), U18.14 (VCC), U19.14 (VCC), U20.14 (VCC), U21.14 (VCC), U22.1 (A->B), U22.20 (VCC), U23.1 (A->B), U23.20 (VCC), U23.8 (A6), U24.1 (A->B), U24.20 (VCC), U25.14 (VCC), U7.14 (VCC), U8.10 (CET), U8.16 (VCC), U8.7 (CEP), U8.9 (~{PE}), U9.16 (VCC), U9.7 (CEP), U9.9 (~{PE}), Y1.14 (Vcc); no longer U1.2 (RDY), U1.36 (BE)
- net A0: now also U22.18 (B0)
- net A1: now also U22.17 (B1)
- net A10: now also U23.16 (B2)
- net A11: now also U23.15 (B3)
- net A12: now also U23.14 (B4)
- net A13: now also U23.13 (B5)
- net A14: now also U6.5, U23.12 (B6), U7.3
- net A15: now also U6.10, U6.4, U23.11 (B7), U7.1
- net A2: now also U22.16 (B2)
- net A3: now also U22.15 (B3)
- net A5: now also U22.13 (B5)
- net A6: now also U22.12 (B6)
- net A7: now also U22.11 (B7)
- net A8: now also U23.18 (B0)
- net A9: now also U23.17 (B1)
- net D0: now also U24.2 (A0)
- net D1: now also U24.3 (A1)
- net D2: now also U24.4 (A2)
- net D3: now also U24.5 (A3)
- net D4: now also U24.6 (A4)
- net D5: now also U24.7 (A5)
- net D6: now also U24.8 (A6)
- net D7: now also U24.9 (A7)
- net GND: now also J7.0, J7.10, J7.5, J7.6, J7.7, J7.8, U10.8 (GND), U11.8 (GND), U12.8 (GND), U13.8 (GND), U14.7 (GND), U15.7 (GND), U16.7 (GND), U17.7 (GND), U18.7 (GND), U19.7 (GND), U20.7 (GND), U21.7 (GND), U22.10 (GND), U23.10 (GND), U23.9 (A7), U24.10 (GND), U25.7 (GND), U7.7 (GND), U8.8 (GND), U9.8 (GND), Y1.7 (GND)
- net ~{IRQ} 1: now also U21.1
- net ~{IRQ} 2: now also U21.2
- net ~{CS}_{VIA B}: now reaches U3.23 (~{CS2})
- net ~{CS}_{VIA B}: now also U7.6
- net VIA Enable: now reaches U3.24 (CS1)
- net VIA Enable: now also U2.24 (CS1), U6.11
- net at U1.4 (~{IRQ}): now also U21.3
- net ~{CS}_{ROM}: now reaches U4.20 (~{CS})
- net ~{CS}_{ROM}: now also U6.6
- net ~{CS}_{VIA A}: now reaches U2.23 (~{CS2})
- net ~{CS}_{VIA A}: now also U22.14 (B4), U7.5
- net ~{CS}_{RAM}: now reaches U5.20 (~{CS})
- net ~{CS}_{RAM}: now also U6.3
- net CLK renamed Clock
- net Clock: now also U6.2, U22.2 (A0), U8.11 (Q3)
- new net: U14.3, U15.3, U16.9, U18.1
- new net: U15.4, U16.2
- new net: U15.6, U17.9
- new net: U16.8, U17.1
- new net: U17.13, U18.6
- new net: U11.1 (~{MR}), U12.1 (~{MR}), U13.1 (~{MR}), U18.8, U19.5
- new net: U10.1 (~{MR}), U11.2 (CP), U12.2 (CP), U13.2 (CP), U15.12, U17.5, U8.1 (~{MR}), U9.1 (~{MR})
- new net: U17.12, U17.8
- new net: U19.12, U19.8
- new net: U15.8, U19.13
- new net: R11.2, U1.2 (RDY)
- new net: U6.1, U7.2
- new net: U6.9, U7.4
- new net: U14.11, U15.9, U16.11, U20.1
- new net: U14.12, U14.8
- new net: U16.10, U19.1
- new net: U14.6, U14.9
- new net: U16.12, U20.4
- new net: U16.3, U20.12
- new net: U16.4, U20.5
- new net: U11.15 (TC), U12.10 (CET)
- new net: U12.15 (TC), U13.10 (CET)
- new net: R6.1, U24.17 (B1)
- new net: J7.1, R5.2, R6.2
- new net: U8.15 (TC), U9.10 (CET)
- new net: U10.10 (CET), U9.15 (TC)
- new net: U10.2 (CP), U8.2 (CP), U9.2 (CP), Y1.8 (OUT)
- new net: R10.1, U24.13 (B5)
- new net: J7.3, R10.2, R9.2
- new net: R9.1, U24.14 (B4)
- new net: R8.1, U24.15 (B3)
- new net: R7.1, U24.16 (B2)
- new net: R5.1, U24.18 (B0)
- new net: U16.6, U20.13
- new net: J7.2, R7.2, R8.2
- new net: U6.12, U6.13, U6.8
- new net: U19.9, U20.6
- new net CPU/~{VGA}: R11.1, U1.36 (BE), U22.19 (CE), U23.19 (CE), U24.19 (CE), U25.3
- new net HBLANK: U17.3, U17.4, U25.1
- new net Q0B: U11.14 (Q0), U18.9
- new net Q1B: U11.13 (Q1), U20.3
- new net Q2B: U11.12 (Q2), U15.10, U16.13, U18.10
- new net Q3B: U11.11 (Q3), U15.11, U18.12, U20.2, U22.9 (A7)
- new net Q4A: U15.5, U18.2, U22.3 (A1), U9.14 (Q0)
- new net Q4B: U12.14 (Q0), U16.5, U23.2 (A0)
- new net Q5A: U15.1, U18.4, U22.4 (A2), U9.13 (Q1)
- new net Q5B: U12.13 (Q1), U14.4, U23.3 (A1)
- new net Q6A: U16.1, U18.5, U22.5 (A3), U9.12 (Q2)
- new net Q6B: U12.12 (Q2), U14.5, U23.4 (A2)
- new net Q7A: U14.1, U22.6 (A4), U9.11 (Q3)
- new net Q7B: U12.11 (Q3), U14.10, U23.5 (A3)
- new net Q8A: U10.14 (Q0), U15.2, U22.7 (A5)
- new net Q8B: U13.14 (Q0), U14.13, U23.6 (A4)
- new net Q9A: U10.13 (Q1), U14.2, U15.13, U22.8 (A6)
- new net Q9B: U13.13 (Q1), U18.13, U23.7 (A5)
- new net VBLANK: U19.3, U19.4, U25.2
- new net ~{HBLANK}: U17.2, U17.6
- new net ~{HSYNC}: J7.13, U17.10, U17.11
- new net ~{VBLANK}: U19.2, U19.6
- new net ~{VSYNC}: J7.14, U19.10, U19.11
- no-connect marks 20 -> 59
Other:
- moved on the sheet: J2, J3, J4, J5, J6, R1, SW1, U1, U2, U3, U4, U5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

Commit message: started working on version 2.0
Parts:
- removed J2, J3, J4, J5: Conn_01x10_Pin, Connector_PinHeader_2.00mm:PinHeader_1x10_P2.00mm_Vertical, symbol Connector:Conn_01x10_Pin
- removed J6: Conn_01x02_Pin, Connector_PinHeader_2.00mm:PinHeader_1x02_P2.00mm_Vertical, symbol Connector:Conn_01x02_Pin
- removed J7: DE15_Socket_HighDensity_MountingHoles, Connector_Dsub:DSUB-15-HD_Socket_Horizontal_P2.29x2.54mm_EdgePinOffset8.35mm_Housed_MountingHolesOffset10.89mm, symbol Connector:DE15_Socket_HighDensity_MountingHoles
- removed R10, R8: 680, Resistor_THT:R_Axial_DIN0207_L6.3mm_D2.5mm_P7.62mm_Horizontal, symbol Device:R
- removed R11: 3.3K, Resistor_THT:R_Axial_DIN0207_L6.3mm_D2.5mm_P7.62mm_Horizontal, symbol Device:R
- removed R9: 1.5K, Resistor_THT:R_Axial_DIN0207_L6.3mm_D2.5mm_P7.62mm_Horizontal, symbol Device:R
- removed U10, U11, U12, U13, U8, U9: 74HC161, Package_DIP:DIP-16_W7.62mm_Socket, symbol 74xx:74LS161
- removed U14, U21: 74LS08, Package_DIP:DIP-14_W7.62mm_Socket, symbol 74xx:74LS08
- removed U15, U20: 74LS10, Package_DIP:DIP-14_W7.62mm_Socket, symbol 74xx:74LS10
- removed U16: 74LS04, Package_DIP:DIP-14_W7.62mm_Socket, symbol 74xx:74LS04
- removed U17, U19: 74LS00, Package_DIP:DIP-14_W7.62mm_Socket, symbol 74xx:74LS00
- removed U18: 74LS20, Package_DIP:DIP-14_W7.62mm_Socket, symbol 74xx:74LS20
- removed U2, U3: W65C22SxP, Package_DIP:DIP-40_W15.24mm_Socket, symbol PCM_65xx-library:W65C22SxP
- removed U22, U23, U24: 74LS245, Package_DIP:DIP-20_W7.62mm_Socket, symbol 74xx:74LS245
- removed U25: 74LS32, Package_DIP:DIP-14_W7.62mm_Socket, symbol 74xx:74LS32
- removed U4: 28C256, Package_DIP:DIP-28_W15.24mm_Socket, symbol Memory_EEPROM:28C256
- removed U5: HM62256BLP, Package_DIP:DIP-28_W15.24mm_Socket, symbol Memory_RAM:HM62256BLP
- removed Y1: 25.175 Mhz, Oscillator:Oscillator_DIP-14, symbol Other:Clock
- added C1, C2, C3, C4, C5, C6, C7: 100nF, Capacitor_SMD:C_0805_2012Metric_Pad1.18x1.45mm_HandSolder, symbol Device:C
- added J2, J3: 2x20 Header, Connector_PinHeader_2.54mm:PinHeader_2x10_P2.54mm_Vertical, symbol Other:Conn_02x10_Odd_Even_Counter_Clockwise_Pin
- added U2: 28C256, Socket:DIP_Socket-28_W11.9mm_W12.7mm_W15.24mm_W17.78mm_W18.5mm_3M_228-1277-00-0602J, symbol Memory_EEPROM:28C256
- added U3: 62256, Package_DIP:DIP-28_W15.24mm_Socket, symbol Memory_RAM:HM62256BLP
- added U4, U5: W65C22S, Package_DIP:DIP-40_W15.24mm_Socket, symbol PCM_65xx-library:W65C22SxP
- added unit 1 of U6
- added unit 5 of U6
- added unit 4 of U6
- added unit 2 of U6
- added unit 6 of U7
- added unit 2 of U7
- added unit 3 of U7
- added unit 7 of U7
- added unit 5 of U7
- added unit 4 of U7
- added U8: 74LS08, Package_DIP:DIP-14_W7.62mm_Socket, symbol 74xx:74LS08
- added U9: 555, Package_DIP:DIP-8_W7.62mm, symbol Timer:NE555P
- R1: value 220 -> 1M; footprint Resistor_THT:R_Axial_DIN0207_L6.3mm_D2.5mm_P7.62mm_Horizontal -> Resistor_SMD:R_0805_2012Metric_Pad1.20x1.40mm_HandSolder
- R2, R3: value 5.11K -> 5K1; footprint Resistor_THT:R_Axial_DIN0207_L6.3mm_D2.5mm_P7.62mm_Horizontal -> Resistor_SMD:R_0805_2012Metric_Pad1.20x1.40mm_HandSolder
- R4: value 1M -> 3K3; footprint Resistor_THT:R_Axial_DIN0207_L6.3mm_D2.5mm_P7.62mm_Horizontal -> Resistor_SMD:R_0805_2012Metric_Pad1.20x1.40mm_HandSolder
- R5, R7: value 1.5K -> 10K; footprint Resistor_THT:R_Axial_DIN0207_L6.3mm_D2.5mm_P7.62mm_Horizontal -> Resistor_SMD:R_0805_2012Metric_Pad1.20x1.40mm_HandSolder
- R6: value 680 -> 1M; footprint Resistor_THT:R_Axial_DIN0207_L6.3mm_D2.5mm_P7.62mm_Horizontal -> Resistor_SMD:R_0805_2012Metric_Pad1.20x1.40mm_HandSolder
- SW1: footprint Button_Switch_THT:SW_PUSH-12mm -> Button_Switch_THT:SW_TH_Tactile_Omron_B3F-100x
- U1: value W65C02SxP -> W65C02
- U6: value 74HC00 -> 74AC00
- U7: value 74HC04 -> 74LS04
Connections:
- net +5V: now also R5.1, R6.1, R7.1, C1.1, C2.1, C3.1, C4.1, C5.1, C6.1, U2.28 (VCC), U3.28 (VCC), U4.20 (VCC), U5.20 (VCC), U9.8 (VCC); no longer R1.1, U1.6 (~{NMI}), U6.14 (VCC), U7.14 (VCC)
- net A0: now also U2.10 (A0), U3.10 (A0), U4.38 (RS0), U5.38 (RS0)
- net A1: now also U2.9 (A1), U3.9 (A1), U4.37 (RS1), U5.37 (RS1)
- net A10: now also U2.21 (A10), U3.21 (A10)
- net A11: now also U2.23 (A11), U3.23 (A11)
- net A12: now also U2.2 (A12), U3.2 (A12)
- net A13: now also U2.26 (A13), U3.26 (A13)
- net A14: now also U2.1 (A14), U3.1 (A14); no longer U6.5, U7.3
- net A15: no longer U6.10, U6.4, U7.1
- net A2: now also U2.8 (A2), U3.8 (A2), U4.36 (RS2), U5.36 (RS2)
- net A3: now also U2.7 (A3), U3.7 (A3), U4.35 (RS3), U5.35 (RS3)
- net A5: now also U2.5 (A5), U3.5 (A5)
- net A6: now also U2.4 (A6), U3.4 (A6)
- net A7: now also U2.3 (A7), U3.3 (A7)
- net A8: now also U2.25 (A8), U3.25 (A8)
- net A9: now also U2.24 (A9), U3.24 (A9)
- net D0: now also U2.11 (D0), U3.11 (Q0), U4.33 (D0), U5.33 (D0)
- net D1: now also U2.12 (D1), U3.12 (Q1), U4.32 (D1), U5.32 (D1)
- net D2: now also U2.13 (D2), U3.13 (Q2), U4.31 (D2), U5.31 (D2)
- net D3: now also U2.15 (D3), U3.15 (Q3), U4.30 (D3), U5.30 (D3)
- net D4: now also U2.16 (D4), U3.16 (Q4), U4.29 (D4), U5.29 (D4)
- net D5: now also U2.17 (D5), U3.17 (Q5), U4.28 (D5), U5.28 (D5)
- net D6: now also U2.18 (D6), U3.18 (Q6), U4.27 (D6), U5.27 (D6)
- net D7: now also U2.19 (D7), U3.19 (Q7), U4.26 (D7), U5.26 (D7)
- net GND: now also R1.2, C1.2, C2.2, C3.2, C4.2, C5.2, C6.2, C7.2, U2.14 (GND), U2.22 (~{OE}), U2.27 (~{WE}), U3.14 (GND), U3.22 (~{OE}), U4.1 (VSS), U5.1 (VSS), U9.1 (GND); no longer R4.2, U6.7 (GND), U7.7 (GND)
- net R/~{W}: now also U3.27 (~{WE})
- net ~{IRQ} 1: now also U5.21 (~{IRQ})
- net ~{IRQ} 2: now also U4.21 (~{IRQ})
- net ~{RES}: now also U4.34 (~{RES}), U5.34 (~{RES}), U9.3 (Q); no longer R1.2, SW1.2
- net at J1.S1 (SHIELD): now also R1.1; no longer R4.1
- net at U1.2 (RDY): now also R4.2
- net ~{IRQ}: now reaches U1.4 (~{IRQ})
- net at U7.2: no longer U6.1
- net at U6.9: no longer U7.4
- net at R6.2: now also C7.1, U9.6 (THR), U9.7 (DIS); no longer R5.2
- net ~{NMI}: now reaches R7.2
- net ~{NMI}: now also U1.6 (~{NMI})
- net CPU/~{VGA}: no longer names the net of U1.36 (BE)
- net CPU/~{VGA}: now also R4.1
- net Clock renamed CLK
- net CLK: no longer U6.2
- removed net VIA Enable: U6.11
- removed net ~{CS}_{RAM}: U6.3
- removed net ~{CS}_{ROM}: U6.6
- net ~{CS}_{VIA A} renamed A4
- net A4: now also U2.6 (A4), U3.6 (A4); no longer U7.5
- removed net ~{CS}_{VIA B}: U7.6
- new net: J3.1, U5.2 (PA0)
- new net: J3.10, U5.14 (PB4)
- new net: J3.11, U5.7 (PA5)
- new net: J3.12, U5.15 (PB5)
- new net: J3.13, U5.8 (PA6)
- new net: J3.14, U5.16 (PB6)
- new net: J3.15, U5.9 (PA7)
- new net: J3.16, U5.17 (PB7)
- new net: J3.17, U5.40 (CA1)
- new net: J3.18, U5.18 (CB1)
- new net: J3.19, U5.39 (CA2)
- new net: J3.2, U5.10 (PB0)
- new net: J3.20, U5.19 (CB2)
- new net: J3.3, U5.3 (PA1)
- new net: J3.4, U5.11 (PB1)
- new net: J3.5, U5.4 (PA2)
- new net: J3.6, U5.12 (PB2)
- new net: J3.7, U5.5 (PA3)
- new net: J3.8, U5.13 (PB3)
- new net: J3.9, U5.6 (PA4)
- new net: J2.2, U4.10 (PB0)
- new net: J2.4, U4.11 (PB1)
- new net: J2.6, U4.12 (PB2)
- new net: J2.8, U4.13 (PB3)
- new net: J2.10, U4.14 (PB4)
- new net: J2.12, U4.15 (PB5)
- new net: J2.14, U4.16 (PB6)
- new net: J2.16, U4.17 (PB7)
- new net: J2.18, U4.18 (CB1)
- new net: J2.20, U4.19 (CB2)
- new net: J2.1, U4.2 (PA0)
- new net: J2.3, U4.3 (PA1)
- new net: J2.19, U4.39 (CA2)
- new net: J2.5, U4.4 (PA2)
- new net: J2.17, U4.40 (CA1)
- new net: J2.7, U4.5 (PA3)
- new net: J2.9, U4.6 (PA4)
- new net: J2.11, U4.7 (PA5)
- new net: J2.13, U4.8 (PA6)
- new net: J2.15, U4.9 (PA7)
- new net: R5.2, SW1.2, U9.2 (TR)
- now unconnected: U6.8
- no-connect marks 59 -> 21
