File: pcb/pcb.kicad_sch (KiCad schematic)
At the start: 27 parts, among them J1 USB_C_Receptacle, J2 2x20 Header, J3 2x20 Header, SW1 SW_Push, U1 W65C02, U2 28C256, U3 62256, U4 W65C22S, U5 W65C22S, U6 74AC00, U7 74LS04, U8 74LS08, U9 555

Commit message: backup
Parts:
- removed C7: 100nF, Capacitor_SMD:C_0805_2012Metric_Pad1.18x1.45mm_HandSolder, symbol Device:C
- removed J1: USB_C_Receptacle, Connector_USB:USB_C_Receptacle_Amphenol_12401548E4-2A, symbol Connector:USB_C_Receptacle
- removed J2, J3: 2x20 Header, Connector_PinHeader_2.54mm:PinHeader_2x10_P2.54mm_Vertical, symbol Other:Conn_02x10_Odd_Even_Counter_Clockwise_Pin
- removed R4: 3K3, Resistor_SMD:R_0805_2012Metric_Pad1.20x1.40mm_HandSolder, symbol Device:R
- removed R6: 1M, Resistor_SMD:R_0805_2012Metric_Pad1.20x1.40mm_HandSolder, symbol Device:R
- removed U2: 28C256, Socket:DIP_Socket-28_W11.9mm_W12.7mm_W15.24mm_W17.78mm_W18.5mm_3M_228-1277-00-0602J, symbol Memory_EEPROM:28C256
- removed U3: 62256, Package_DIP:DIP-28_W15.24mm_Socket, symbol Memory_RAM:HM62256BLP
- removed U5: W65C22S, Package_DIP:DIP-40_W15.24mm_Socket, symbol PCM_65xx-library:W65C22SxP
- removed U6: 74AC00, Package_DIP:DIP-14_W7.62mm_Socket, symbol 74xx:74LS00
- removed U7: 74LS04, Package_DIP:DIP-14_W7.62mm_Socket, symbol 74xx:74LS04
- removed U8: 74LS08, Package_DIP:DIP-14_W7.62mm_Socket, symbol 74xx:74LS08
- removed U9: 555, Package_DIP:DIP-8_W7.62mm, symbol Timer:NE555P
- added C1, C11, C12, C13, C14, C15, C16, C3, C9: 0.1uF, Capacitor_SMD:C_0805_2012Metric, symbol Device:C
- added C5: 10uF, Capacitor_THT:C_Radial_D5.0mm_H7.0mm_P2.00mm, symbol Device:C_Polarized_US
- added D1: D, symbol Device:D
- added H1, H2, H3, H4: MountingHole_Pad, MountingHole:MountingHole_3.2mm_M3_Pad, symbol Mechanical:MountingHole_Pad
- added J1: USB_C_Receptacle_USB2.0_16P, Connector_USB:USB_C_Receptacle_GCT_USB4085, symbol Connector:USB_C_Receptacle_USB2.0_16P
- added J2: VGA Connector, Connector_Dsub:DSUB-15-HD_Socket_Horizontal_P2.29x2.54mm_EdgePinOffset8.35mm_Housed_MountingHolesOffset10.89mm, symbol Connector:DE15_Socket_HighDensity_MountingHoles
- added J3: 2x11 Header, Connector_IDC:IDC-Header_2x11_P2.54mm_Horizontal, symbol Other:Conn_02x11_Odd_Even_Counter_Clockwise_Pin
- added J4: 2x03 Header, Connector_IDC:IDC-Header_2x03_P2.54mm_Horizontal, symbol Other:Conn_02x03_Odd_Even_Counter_Clockwise_Pin_1
- added J5: 2x17 Header, Connector_IDC:IDC-Header_2x20_P2.54mm_Horizontal, symbol Other:Conn_02x20_Odd_Even_Pin
- added R24, R5, R7: 3K3, Resistor_SMD:R_0805_2012Metric, symbol Device:R
- added U1: 74AC154, Package_SO:SOIC-24W_7.5x15.4mm_P1.27mm, symbol 74xx:74LS154
- added U10: SST39SF010, Package_LCC:PLCC-32_THT-Socket, symbol Memory_Flash:SST39SF010
- added U11: W65C51NxP, Package_DIP:DIP-28_W15.24mm_Socket, symbol PCM_65xx-library:W65C51NxP
- added U12, U13, U14: 74AC245, Package_SO:TSSOP-20_4.4x6.5mm_P0.65mm, symbol 74xx:74LS245
- added U2: 74AC138, Package_SO:SOIC-16_3.9x9.9mm_P1.27mm, symbol 74xx:74LS138
- added U3: 74AC11, Package_SO:SOIC-14_3.9x8.7mm_P1.27mm, symbol 74xx:74LS11
- added U4: 74AC238, Package_SO:SOIC-16_3.9x9.9mm_P1.27mm, symbol 74xx:74HC238
- added U6: AS7C256C, Package_DIP:DIP-28_W7.62mm_Socket, symbol Other:AS7C256C
- added U7, U9: 7005, Package_QFP:TQFP-64_14x14mm_P0.8mm, symbol Other:7005
- added Y1: 8MHz, Oscillator:Oscillator_SMD_SeikoEpson_SG8002CA-4Pin_7.0x5.0mm, symbol Other:Oscillator_Clock
- added Y2: 1.8432MHz, Oscillator:Oscillator_SMD_SeikoEpson_SG8002CA-4Pin_7.0x5.0mm, symbol Other:Oscillator_Clock
- C10: renamed from C5; value 100nF -> 0.1uF; footprint Capacitor_SMD:C_0805_2012Metric_Pad1.18x1.45mm_HandSolder -> Capacitor_SMD:C_0805_2012Metric
- C2, C4, C6: value 100nF -> 0.1uF; footprint Capacitor_SMD:C_0805_2012Metric_Pad1.18x1.45mm_HandSolder -> Capacitor_SMD:C_0805_2012Metric
- C7: renamed from C1; value 100nF -> 0.1uF; footprint Capacitor_SMD:C_0805_2012Metric_Pad1.18x1.45mm_HandSolder -> Capacitor_SMD:C_0805_2012Metric
- C8: renamed from C3; value 100nF -> 0.1uF; footprint Capacitor_SMD:C_0805_2012Metric_Pad1.18x1.45mm_HandSolder -> Capacitor_SMD:C_0805_2012Metric
- R1, R2, R3: footprint Resistor_SMD:R_0805_2012Metric_Pad1.20x1.40mm_HandSolder -> Resistor_SMD:R_0805_2012Metric
- R4: renamed from R5; footprint Resistor_SMD:R_0805_2012Metric_Pad1.20x1.40mm_HandSolder -> Resistor_SMD:R_0805_2012Metric
- R6: renamed from R7; value 10K -> 3K3; footprint Resistor_SMD:R_0805_2012Metric_Pad1.20x1.40mm_HandSolder -> Resistor_SMD:R_0805_2012Metric
- SW1: footprint Button_Switch_THT:SW_TH_Tactile_Omron_B3F-100x -> Button_Switch_THT:SW_PUSH_6mm
- renumbered U1 to U5, U4 to U8
Connections:
- net A0: now also U10.12 (A0), U11.13 (RS0), U12.2 (A0), U6.10 (A0), U7.44 (A_{0L}), U9.37 (A_{0R})
- net A1: now also U10.11 (A1), U11.14 (RS1), U14.9 (A7), U6.9 (A1), U7.45 (A_{1L}), U9.36 (A_{1R})
- net A10: now also U10.23 (A10), U12.7 (A5), U6.21 (A10), U7.54 (A_{10L}), U9.27 (A_{10R})
- net A11: now also U10.25 (A11), U14.4 (A2), U6.23 (A11), U7.55 (A_{11L}), U9.26 (A_{11R})
- net A12: now also U1.23 (A0), U10.4 (A12), U12.8 (A6), U6.2 (A12), U7.56 (A_{12L})
- net A13: now also U1.22 (A1), U10.28 (A13), U14.3 (A1), U2.1 (A0), U6.26 (A13)
- net A14: now also U1.21 (A2), U12.9 (A7), U2.2 (A1), U6.1 (A14)
- net A15: now also U1.20 (A3), U14.2 (A0), U2.3 (A2)
- net A2: now also U10.10 (A2), U12.3 (A1), U6.8 (A2), U7.46 (A_{2L}), U9.35 (A_{2R})
- net A3: now also U10.9 (A3), U14.8 (A6), U6.7 (A3), U7.47 (A_{3L}), U9.34 (A_{3R})
- net A4: now also U10.8 (A4), U12.4 (A2), U4.1 (A0), U6.6 (A4), U7.48 (A_{4L}), U9.33 (A_{4R})
- net A5: now also U10.7 (A5), U14.7 (A5), U4.2 (A1), U6.5 (A5), U7.49 (A_{5L}), U9.32 (A_{5R})
- net A6: now also U10.6 (A6), U12.5 (A3), U4.3 (A2), U6.4 (A6), U7.50 (A_{6L}), U9.31 (A_{6R})
- net A7: now also U10.5 (A7), U14.6 (A4), U6.3 (A7), U7.51 (A_{7L}), U9.30 (A_{7R})
- net A8: now also U10.27 (A8), U12.6 (A4), U6.25 (A8), U7.52 (A_{8L}), U9.29 (A_{8R})
- net A9: now also U10.26 (A9), U14.5 (A3), U6.24 (A9), U7.53 (A_{9L}), U9.28 (A_{9R})
- net CLK: now also U5.39 (ϕ2), U8.25 (ϕ2), J5.32, U11.27 (ϕ2); no longer U5.37 (ϕ0)
- net D0: now also U10.13 (D0), U11.18 (D0), U13.11 (B7), U6.11 (Q0), U7.63 (I/O_{0L}), U9.10 (I/O_{0R})
- net D1: now also U10.14 (D1), U11.19 (D1), U13.12 (B6), U6.12 (Q1), U7.64 (I/O_{1L}), U9.11 (I/O_{1R})
- net D2: now also U10.15 (D2), U11.20 (D2), U13.13 (B5), U6.13 (Q2), U7.1 (I/O_{2L}), U9.12 (I/O_{2R})
- net D3: now also U10.17 (D3), U11.21 (D3), U13.14 (B4), U6.15 (Q3), U7.2 (I/O_{3L}), U9.14 (I/O_{3R})
- net D4: now also U10.18 (D4), U11.22 (D4), U13.15 (B3), U6.16 (Q4), U7.3 (I/O_{4L}), U9.15 (I/O_{4R})
- net D5: now also U10.19 (D5), U11.23 (D5), U13.16 (B2), U6.17 (Q5), U7.4 (I/O_{5L}), U9.16 (I/O_{5R})
- net D6: now also U10.20 (D6), U11.24 (D6), U13.17 (B1), U6.18 (Q6), U7.6 (I/O_{6L}), U9.17 (I/O_{6R})
- net D7: now also U10.21 (D7), U11.25 (D7), U13.18 (B0), U6.19 (Q7), U7.7 (I/O_{7L}), U9.18 (I/O_{7R})
- net GND: now also C6.1, C1.2, C11.2, C12.2, C13.2, C14.2, C15.2, C16.1, C3.2, C5.2, C9.2, H1.1, H2.1, H3.1, H4.1, J1.A1 (GND), J1.A12 (GND), J1.B1 (GND), J1.B12 (GND), J2.0, J2.10, J2.5, J2.6, J2.7, J2.8, J3.2, J4.6, J5.28, J5.29, J5.30, J5.33, J5.34, J5.37, J5.38, U1.12 (GND), U1.18 (E0), U1.19 (E1), U10.16 (GND), U10.2 (A16), U10.24 (OE), U10.29 (A14), U10.3 (A15), U11.1 (VSS), U12.10 (GND), U13.10 (GND), U14.10 (GND), U2.4 (E1), U2.5 (E2), U2.8 (GND), U3.7 (GND), U4.4 (~{E1}), U4.5 (~{E2}), U4.8 (GND), U6.14 (GND), U6.22 (~{OE}), U7.19 (~{OE}_{R}), U7.22 (~{CE}_{R}), U7.24 (GND), U7.41 (GND), U7.5 (GND), U7.62 (~{OE}_{L}), U7.9 (GND), U9.19 (~{OE}_{R}), U9.22 (~{CE}_{R}), U9.24 (GND), U9.41 (GND), U9.5 (GND), U9.62 (~{OE}_{L}), U9.9 (GND), Y1.2 (GND), Y2.2 (GND); no longer C6.2
- net R/~{W}: now also U8.22 (R/~{W}), J5.27, U11.28 (R/~{W}), U13.1 (A->B), U6.27 (~{WE}), U7.61 (R/~{W}_{L}), U9.61 (R/~{W}_{L})
- net ~{IRQ}: now also D1.2 (A), J5.31, R5.1
- net ~{NMI}: now also R6.1, J5.35; no longer R6.2
- net ~{RES}: now also C6.2, R4.2, SW1.2, J5.39, U11.4 (~{RES})
- net at R2.1: now also J1.B5 (CC2)
- net at U8.10 (PB0): now also J3.22
- net at U8.11 (PB1): now also J3.20
- net at U8.12 (PB2): now also J3.18
- net at U8.13 (PB3): now also J3.16
- net at U8.14 (PB4): now also J3.14
- net at U8.15 (PB5): now also J3.12
- net at U8.16 (PB6): now also J3.10
- net at U8.17 (PB7): now also J3.8
- net at U8.18 (CB1): now also J3.6
- net at U8.19 (CB2): now also J3.4
- net at U8.2 (PA0): now also J3.17
- net ~{CS}_{IO}: now reaches U8.23 (~{CS2})
- net ~{CS}_{IO}: now also U1.8 (S7), U11.3 (~{CS2})
- net CS_{VIA}: now reaches U8.24 (CS1)
- net CS_{VIA}: now also U4.15 (Y0)
- net at U8.3 (PA1): now also J3.15
- net at U8.39 (CA2): now also J3.19
- net at U8.4 (PA2): now also J3.13
- net at U8.40 (CA1): now also J3.21
- net at U8.5 (PA3): now also J3.11
- net at U8.6 (PA4): now also J3.9
- net at U8.7 (PA5): now also J3.7
- net at U8.8 (PA6): now also J3.5
- net at U8.9 (PA7): now also J3.3
- net at R1.1: now also J1.S1 (SHIELD)
- net VCC: now reaches U5.36 (BE)
- net VCC: now also C10.1, C2.1, C4.1, C7.1, C8.1, R4.1, R6.2, U5.38 (~{SO}), U5.8 (VDD), U8.20 (VCC), C1.1, C11.1, C12.1, C13.1, C14.1, C15.1, C16.2, C3.1, C5.1, C9.1, J1.A4 (VBUS), J1.A9 (VBUS), J1.B4 (VBUS), J1.B9 (VBUS), J3.1, J4.1, J5.1, J5.2, R24.1, R5.2, R7.2, U1.24 (VCC), U10.31 (PGM), U10.32 (VCC), U11.15 (VCC), U12.1 (A->B), U12.20 (VCC), U13.20 (VCC), U14.1 (A->B), U14.20 (VCC), U2.16 (VCC), U2.6 (E3), U3.13, U3.14 (VCC), U4.16 (VCC), U4.6 (E3), U6.28 (VCC), U7.13 (VCC), U7.20 (R/~{W}_{R}), U7.21 (~{SEM}_{R}), U7.40 (M/~{S}), U7.57 (VCC), U7.60 (~{SEM}_{L}), U7.8 (VCC), U9.13 (VCC), U9.20 (R/~{W}_{R}), U9.21 (~{SEM}_{R}), U9.40 (M/~{S}), U9.57 (VCC), U9.60 (~{SEM}_{L}), U9.8 (VCC), Y1.1 (EOH), Y1.4 (VCC), Y2.1 (EOH), Y2.4 (VCC)
- net RDY: now reaches U5.2 (RDY)
- net RDY: now also J5.40, R7.1
- net SYNC: now reaches U5.7 (SYNC)
- net SYNC: now also J5.36
- net at R3.1: now also J1.A5 (CC1)
- removed net +5V: C10.1, C2.1, C4.1, C6.1, C7.1, C8.1, R4.1, R6.1, U5.38 (~{SO}), U5.8 (VDD), U8.20 (VCC)
- net ~{IRQ} 2 renamed ~{IRQ}_{VIA}
- net ~{IRQ}_{VIA}: now also U3.11
- new net: U2.10 (O5), U3.3
- new net: U2.9 (O6), U3.4
- new net: U2.7 (O7), U3.5
- new net: J5.26, U13.2 (A0)
- new net: J5.25, U13.3 (A1)
- new net: J5.24, U13.4 (A2)
- new net: J5.23, U13.5 (A3)
- new net: J5.22, U13.6 (A4)
- new net: J5.21, U13.7 (A5)
- new net: J5.20, U13.8 (A6)
- new net: J5.19, U13.9 (A7)
- new net: U5.37 (ϕ0), Y1.3 (OUT)
- new net: U11.6 (XTAL1), Y2.3 (OUT)
- new net: D1.1 (K), U3.8
- new net: U2.15 (O0), U3.1
- new net: U2.14 (O1), U3.2
- new net: J5.10, U14.14 (B4)
- new net: J5.11, U12.14 (B4)
- new net: J5.12, U14.15 (B3)
- new net: J5.13, U12.13 (B5)
- new net: J5.14, U14.16 (B2)
- new net: J5.15, U12.12 (B6)
- new net: J5.16, U14.17 (B1)
- new net: J5.17, U12.11 (B7)
- new net: J5.18, U14.18 (B0)
- new net: J5.3, U12.18 (B0)
- new net: J5.4, U14.11 (B7)
- new net: J5.5, U12.17 (B1)
- new net: J5.6, U14.12 (B6)
- new net: J5.7, U12.16 (B2)
- new net: J5.8, U14.13 (B5)
- new net: J5.9, U12.15 (B3)
- new net: J4.2, U11.12 (RxD)
- new net: J4.3, U11.8 (~{RTS})
- new net: J4.4, U11.10 (TxD)
- new net: J4.5, U11.9 (~{CTS})
- new net CS_{ACIA}: U11.2 (CS1), U4.14 (Y1)
- new net CS_{PPU}: U4.13 (Y2)
- new net PPU/B: J2.3
- new net PPU/G: J2.2
- new net PPU/R: J2.1
- new net PPU/TS_{CPU}: U9.25 (A_{12R})
- new net PPU/~{HSYNC}: J2.13
- new net PPU/~{VSYNC}: J2.14
- new net TMA0: U9.44 (A_{0L})
- new net TMA1: U9.45 (A_{1L})
- new net TMA10: U9.54 (A_{10L})
- new net TMA11: U9.55 (A_{11L})
- new net TMA12: U9.56 (A_{12L})
- new net TMA2: U9.46 (A_{2L})
- new net TMA3: U9.47 (A_{3L})
- new net TMA4: U9.48 (A_{4L})
- new net TMA5: U9.49 (A_{5L})
- new net TMA6: U9.50 (A_{6L})
- new net TMA7: U9.51 (A_{7L})
- new net TMA8: U9.52 (A_{8L})
- new net TMA9: U9.53 (A_{9L})
- new net TMD0: U9.7 (I/O_{7L})
- new net TMD1: U9.6 (I/O_{6L})
- new net TMD2: U9.4 (I/O_{5L})
- new net TMD3: U9.3 (I/O_{4L})
- new net TMD4: U9.2 (I/O_{3L})
- new net TMD5: U9.1 (I/O_{2L})
- new net TMD6: U9.64 (I/O_{1L})
- new net TMD7: U9.63 (I/O_{0L})
- new net VMA0: U7.37 (A_{0R})
- new net VMA1: U7.36 (A_{1R})
- new net VMA10: U7.27 (A_{10R})
- new net VMA11: U7.26 (A_{11R})
- new net VMA12: U7.25 (A_{12R})
- new net VMA2: U7.35 (A_{2R})
- new net VMA3: U7.34 (A_{3R})
- new net VMA4: U7.33 (A_{4R})
- new net VMA5: U7.32 (A_{5R})
- new net VMA6: U7.31 (A_{6R})
- new net VMA7: U7.30 (A_{7R})
- new net VMA8: U7.29 (A_{8R})
- new net VMA9: U7.28 (A_{9R})
- new net VMD0: U7.10 (I/O_{0R})
- new net VMD1: U7.11 (I/O_{1R})
- new net VMD2: U7.12 (I/O_{2R})
- new net VMD3: U7.14 (I/O_{3R})
- new net VMD4: U7.15 (I/O_{4R})
- new net VMD5: U7.16 (I/O_{5R})
- new net VMD6: U7.17 (I/O_{6R})
- new net VMD7: U7.18 (I/O_{7R})
- new net ~{CS}_{EXP}: U12.19 (CE), U13.19 (CE), U14.19 (CE), U2.11 (O4)
- new net ~{CS}_{RAM}: U3.12, U6.20 (~{CS})
- new net ~{CS}_{ROM}: U10.22 (CE), U3.6
- new net ~{CS}_{TM}: U1.7 (S6), U9.59 (~{CE}_{L})
- new net ~{CS}_{VRAM}: U2.13 (O2), U7.59 (~{CE}_{L})
- new net ~{IRQ}_{ACIA}: R24.2, U11.26 (~{IRQ}), U3.10
- new net ~{IRQ}_{PPU}: U3.9
- no-connect marks 21 -> 49
Other:
- added sheet PPU (PPU.kicad_sch)
- moved on the sheet: C10, C7, C8, R4, R6, SW1, U5, U8
